File: hardware/accessories/filters/filters.sch (KiCad schematic (older format))
At the start: 34 parts

Commit message: get filter pcb
Parts:
- added C11, C12: 10u, Capacitor_SMD:C_1206_3216Metric_Pad1.42x1.75mm_HandSolder, symbol Device:C_Small
- added C13, C14: 100n, Capacitor_SMD:C_0603_1608Metric_Pad1.05x0.95mm_HandSolder, symbol Device:C_Small
- added J5: PWR, Connector_PinHeader_2.54mm:PinHeader_1x02_P2.54mm_Vertical, symbol Connector:Conn_01x02_Male
- C1, C2, C3, C4, C5, C6, C7, C8: renamed from C?; footprint (none) -> Capacitor_SMD:C_0603_1608Metric_Pad1.05x0.95mm_HandSolder
- C10, C9: renamed from C?; footprint (none) -> Capacitor_SMD:C_1206_3216Metric_Pad1.42x1.75mm_HandSolder
- J1, J2, J3, J4: renamed from J?; footprint (none) -> Connector_Coaxial:U.FL_Hirose_U.FL-R-SMT-1_Vertical
- R1, R10, R11, R12, R13, R14, R15, R2, R3, R4, R5, R6, R7, R8: renamed from R?; footprint (none) -> Resistor_SMD:R_0603_1608Metric_Pad1.05x0.95mm_HandSolder
- U1: renamed from U?; value LM833 -> ada4891-2; footprint (none) -> Package_SO:MSOP-8_3x3mm_P0.65mm
- U2: renamed from U?; footprint (none) -> Package_SO:MSOP-8_3x3mm_P0.65mm
Connections:
- net GND: now also C11.2, C12.2, C13.1, C14.1, J5.2 (Pin_2); no longer C7.1, C8.1, R14.2, R15.2, U1.6 (-), U1.7, U2.6 (-), U2.7
- net VCC: now also C11.1, C12.1, C13.2, C14.2, J5.1 (Pin_1)
- new net: C7.1, R14.2, U1.6 (-), U1.7
- new net: C8.1, R15.2, U2.6 (-), U2.7
Other:
- note added: "Text: R C value need to be adj"

Commit message: update the filter sch
Parts:
- C1, C2: value 150p -> 120p
- C3, C4: value 120p -> 100p
- C5, C6: value 56p -> 47p
- C7, C8: value 390p -> 330p
- R10, R11: value 9.5k -> 2.2k
- R12, R13: value 12k -> 3k
- R5, R6: value 9.1k -> 2.4k
- R7, R8: value 15k -> 3.3k
Other:
- note added: "500k, 4th order Butterworth"
- note removed: "100k, 4th order Butterworth"
Changed lines of the file:
@@
 EESchema Schematic File Version 4
+LIBS:filters-cache
 EELAYER 26 0
 EELAYER END
@@
 P 3600 1650
 F 0 "R7" V 3395 1650 50  0000 C CNN
-F 1 "15k" V 3486 1650 50  0000 C CNN
+F 1 "3.3k" V 3486 1650 50  0000 C CNN
 F 2 "Resistor_SMD:R_0603_1608Metric_Pad1.05x0.95mm_HandSolder" V 3640 1640 50  0001 C CNN
 F 3 "~" H 3600 1650 50  0001 C CNN
@@
 P 3050 1650
 F 0 "R5" V 2845 1650 50  0000 C CNN
-F 1 "9.1k" V 2936 1650 50  0000 C CNN
+F 1 "2.4k" V 2936 1650 50  0000 C CNN
 F 2 "Resistor_SMD:R_0603_1608Metric_Pad1.05x0.95mm_HandSolder" V 3090 1640 50  0001 C CNN
 F 3 "~" H 3050 1650 50  0001 C CNN
@@
 P 3900 2000
 F 0 "C3" H 3992 2046 50  0000 L CNN
-F 1 "120p" H 3992 1955 50  0000 L CNN
+F 1 "100p" H 3992 1955 50  0000 L CNN
 F 2 "Capacitor_SMD:C_0603_1608Metric_Pad1.05x0.95mm_HandSolder" H 3900 2000 50  0001 C CNN
 F 3 "~" H 3900 2000 50  0001 C CNN
@@
 P 3700 1100
 F 0 "C1" V 3471 1100 50  0000 C CNN
-F 1 "150p" V 3562 1100 50  0000 C CNN
+F 1 "120p" V 3562 1100 50  0000 C CNN
 F 2 "Capacitor_SMD:C_0603_1608Metric_Pad1.05x0.95mm_HandSolder" H 3700 1100 50  0001 C CNN
 F 3 "~" H 3700 1100 50  0001 C CNN
@@
 P 5000 1750
 F 0 "R10" V 4795 1750 50  0000 C CNN
-F 1 "9.5k" V 4886 1750 50  0000 C CNN
+F 1 "2.2k" V 4886 1750 50  0000 C CNN
 F 2 "Resistor_SMD:R_0603_1608Metric_Pad1.05x0.95mm_HandSolder" V 5040 1740 50  0001 C CNN
 F 3 "~" H 5000 1750 50  0001 C CNN
@@
 P 5600 1750
 F 0 "R12" V 5395 1750 50  0000 C CNN
-F 1 "12k" V 5486 1750 50  0000 C CNN
+F 1 "3k" V 5486 1750 50  0000 C CNN
 F 2 "Resistor_SMD:R_0603_1608Metric_Pad1.05x0.95mm_HandSolder" V 5640 1740 50  0001 C CNN
 F 3 "~" H 5600 1750 50  0001 C CNN
@@
 P 5800 2000
 F 0 "C5" H 5600 2000 50  0000 L CNN
-F 1 "56p" H 5600 1900 50  0000 L CNN
+F 1 "47p" H 5600 1900 50  0000 L CNN
 F 2 "Capacitor_SMD:C_0603_1608Metric_Pad1.05x0.95mm_HandSolder" H 5800 2000 50  0001 C CNN
 F 3 "~" H 5800 2000 50  0001 C CNN
@@
 P 5900 1100
 F 0 "C7" V 5671 1100 50  0000 C CNN
-F 1 "390p" V 5762 1100 50  0000 C CNN
+F 1 "330p" V 5762 1100 50  0000 C CNN
 F 2 "Capacitor_SMD:C_0603_1608Metric_Pad1.05x0.95mm_HandSolder" H 5900 1100 50  0001 C CNN
 F 3 "~" H 5900 1100 50  0001 C CNN
@@
 	1600 1950 1600 1850
 Text Notes 4600 950  0    50   ~ 0
-100k, 4th order Butterworth
+500k, 4th order Butterworth
 $Comp
 L Amplifier_Operational:LM358 U2
@@
 P 3650 3700
 F 0 "R8" V 3445 3700 50  0000 C CNN
-F 1 "15k" V 3536 3700 50  0000 C CNN
+F 1 "3.3k" V 3536 3700 50  0000 C CNN
 F 2 "Resistor_SMD:R_0603_1608Metric_Pad1.05x0.95mm_HandSolder" V 3690 3690 50  0001 C CNN
 F 3 "~" H 3650 3700 50  0001 C CNN
@@
 P 3100 3700
 F 0 "R6" V 2895 3700 50  0000 C CNN
-F 1 "9.1k" V 2986 3700 50  0000 C CNN
+F 1 "2.4k" V 2986 3700 50  0000 C CNN
 F 2 "Resistor_SMD:R_0603_1608Metric_Pad1.05x0.95mm_HandSolder" V 3140 3690 50  0001 C CNN
 F 3 "~" H 3100 3700 50  0001 C CNN
@@
 P 3950 4050
 F 0 "C4" H 4042 4096 50  0000 L CNN
-F 1 "120p" H 4042 4005 50  0000 L CNN
+F 1 "100p" H 4042 4005 50  0000 L CNN
 F 2 "Capacitor_SMD:C_0603_1608Metric_Pad1.05x0.95mm_HandSolder" H 3950 4050 50  0001 C CNN
 F 3 "~" H 3950 4050 50  0001 C CNN
@@
 P 3750 3150
 F 0 "C2" V 3521 3150 50  0000 C CNN
-F 1 "150p" V 3612 3150 50  0000 C CNN
+F 1 "120p" V 3612 3150 50  0000 C CNN
 F 2 "Capacitor_SMD:C_0603_1608Metric_Pad1.05x0.95mm_HandSolder" H 3750 3150 50  0001 C CNN
 F 3 "~" H 3750 3150 50  0001 C CNN
@@
 P 5050 3800
 F 0 "R11" V 4845 3800 50  0000 C CNN
-F 1 "9.5k" V 4936 3800 50  0000 C CNN
+F 1 "2.2k" V 4936 3800 50  0000 C CNN
 F 2 "Resistor_SMD:R_0603_1608Metric_Pad1.05x0.95mm_HandSolder" V 5090 3790 50  0001 C CNN
 F 3 "~" H 5050 3800 50  0001 C CNN
@@
 P 5650 3800
 F 0 "R13" V 5445 3800 50  0000 C CNN
-F 1 "12k" V 5536 3800 50  0000 C CNN
+F 1 "3k" V 5536 3800 50  0000 C CNN
 F 2 "Resistor_SMD:R_0603_1608Metric_Pad1.05x0.95mm_HandSolder" V 5690 3790 50  0001 C CNN
 F 3 "~" H 5650 3800 50  0001 C CNN
@@
 P 5850 4050
 F 0 "C6" H 5650 4050 50  0000 L CNN
-F 1 "56p" H 5650 3950 50  0000 L CNN
+F 1 "47p" H 5650 3950 50  0000 L CNN
 F 2 "Capacitor_SMD:C_0603_1608Metric_Pad1.05x0.95mm_HandSolder" H 5850 4050 50  0001 C CNN
 F 3 "~" H 5850 4050 50  0001 C CNN
@@
 P 5950 3150
 F 0 "C8" V 5721 3150 50  0000 C CNN
-F 1 "390p" V 5812 3150 50  0000 C CNN
+F 1 "330p" V 5812 3150 50  0000 C CNN
 F 2 "Capacitor_SMD:C_0603_1608Metric_Pad1.05x0.95mm_HandSolder" H 5950 3150 50  0001 C CNN
 F 3 "~" H 5950 3150 50  0001 C CNN
