File: hardware/accessories/filters/filters.kicad_pcb (KiCad board)
At the start: 2 copper layers, 35 parts, among them J1 Conn_Coaxial, J2 Conn_Coaxial, J3 Conn_Coaxial, J4 Conn_Coaxial, J5 PWR, U1 ada4891-2, U2 ada4891-2

Commit message: Update filters.kicad_pcb
Parts:
- moved C8 8.32 mm to (144.5, 108.0), turned to 270 degrees
- moved C7 7.37 mm to (146.1, 85.3), turned to 90 degrees
- moved R13 3.84 mm to (146.6, 108.0), turned to 270 degrees
- moved R12 3.58 mm to (144.0, 85.3), turned to 90 degrees
- moved R11 2.09 mm to (148.6, 108.0), turned to 90 degrees
- moved R10 1.28 mm to (141.7, 85.3), turned to 270 degrees
Routing:
- net Net-(C8-Pad2): track 17.0 -> 4.06 mm
- net Net-(C7-Pad2): track 14.8 -> 4.32 mm
- net Net-(C8-Pad1): track 11.5 -> 16.3 mm
- net Net-(C7-Pad1): track 7.49 -> 11.9 mm
- net Net-(C6-Pad1): track 11.2 -> 9.30 mm
- net Net-(C5-Pad1): track 9.92 -> 8.57 mm
Other:
- net class Default: trace_width 0.25 -> 0.45
